File: ch32v203_TestBoard/ch32v203_TestBoard.kicad_pcb (KiCad board)
At the start: 2 copper layers, 100 x 100 mm, 31 parts, among them J5 Conn_01x06, J6 USB_B, J7 Barrel_Jack_Switch, J8 Conn_01x03_Pin, U1 CH32V203K8T6, U2 AZ1117-3.3, Y1 Crystal_GND2

Commit message: 一部修正
Parts:
- J1: renamed from PB; footprint Connector_PinSocket_2.54mm:PinSocket_1x08_P2.54mm_Vertical -> Connector_PinHeader_2.54mm:PinHeader_1x08_P2.54mm_Vertical
- J12: renamed from POWER; footprint Connector_PinSocket_2.54mm:PinSocket_1x04_P2.54mm_Vertical -> Connector_PinHeader_2.54mm:PinHeader_1x04_P2.54mm_Vertical
- J4: renamed from ADC; footprint Connector_PinSocket_2.54mm:PinSocket_1x10_P2.54mm_Vertical -> Connector_PinHeader_2.54mm:PinHeader_1x10_P2.54mm_Vertical
- J5: value Conn_01x06 -> WRITER
- moved D5 0.06 mm to (178.0, 57.1)
- renumbered SPI to J10, I2C to J11, PA to J2, PD to J3, UART to J9, RESET to SW1, BOOT to SW2
Connections:
- J5 pad 1: +5V -> Net-(D5-A)
Routing:
- net +5V: track 177.3 -> 154.5 mm
- net Net-(D5-A): track 9.31 -> 31.6 mm, vias 0 -> 1
- net Net-(J1-Pin_2): track 92.2 -> 79.4 mm, vias 5 -> 3
- net +3.3V: track 54.9 -> 44.3 mm, vias 3 -> 2
- net Net-(J1-Pin_1): track 80.1 -> 84.5 mm
- net Net-(D1-K): track 6.76 -> 7.29 mm
- net Net-(J8-Pin_2): track 29.0 -> 29.1 mm, vias 0 -> 3
- net NRST: vias 5 -> 4
- net GND: vias 4 -> 2
